File: ECE4450_FinalProject/ECE4450_FinalProject.kicad_pcb (KiCad board)
At the start: 2 copper layers, 75 x 100 mm, 19 parts, among them J1 PWR, J2 IN, J3 OUT, P1 Front_panel, Q1 BS250, U1 MAX1044, U2 SSM2164PZ, U3 TL072

Commit message: Commit test
Parts:
- moved U2 24.4 mm to (62.0, 58.4)
Changed lines of the file:
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@@
 	(footprint "SSM2164:N_16_ADI"
 		(layer "F.Cu")
-		(at 62 82.8)
+		(at 62 58.42)
 		(tags "SSM2164PZ ")
 		(property "Reference" "U2"

Commit message: commit test
Parts:
- moved U2 17.3 mm to (45.0, 61.2)
Changed lines of the file:
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@@
 	(footprint "SSM2164:N_16_ADI"
 		(layer "F.Cu")
-		(at 62 58.42)
+		(at 44.958 61.214)
 		(tags "SSM2164PZ ")
 		(property "Reference" "U2"

Commit message: layout and single trace lacer
Parts:
- removed C2, C3: 0u1, Aaron_Library:C_Axial_Aaron
- removed P1: Front_panel, Aaron_Library:Potentiometer_TW_Frontpanel
- removed TP1: In_a_row, Potentiometer_THT:Potentiometer_Bourns_3296W_Vertical
- removed TP2: In_a_triangle, Aaron_Library:Potentiometer_Square_Trimpot_Aaron
- added C10: 220p, Aaron_Library:C_Axial_Aaron, F.Cu at (45.7, 84.1)
- added C11: 1500p, Aaron_Library:C_Axial_Aaron, F.Cu at (40.6, 62.2)
- added C12: 1500p, Aaron_Library:C_Axial_Aaron, F.Cu at (72.4, 69.8)
- added C13: 220p, Aaron_Library:C_Axial_Aaron, F.Cu at (101.4, 49.7)
- added C14: 1500p, Aaron_Library:C_Axial_Aaron, F.Cu at (50.8, 62.1)
- added C15: 220p, Aaron_Library:C_Axial_Aaron, F.Cu at (33.0, 78.7)
- added C16: 1u, Aaron_Library:C_Axial_Aaron, F.Cu at (43.1, 116.8)
- added C17: 3.6p, Aaron_Library:C_Axial_Aaron, F.Cu at (35.6, 114.3)
- added C18: 3.6p, Aaron_Library:C_Axial_Aaron, F.Cu at (33.0, 83.9)
- added C5: 100p, Aaron_Library:C_Axial_Aaron, F.Cu at (63.4, 118.1)
- added C6: 2200p, Aaron_Library:C_Axial_Aaron, F.Cu at (38.1, 41.9)
- added C9: 220p, Aaron_Library:C_Axial_Aaron, F.Cu at (30.5, 62.1)
- added D1: 1N4148, Diode_THT:D_DO-35_SOD27_P7.62mm_Horizontal, F.Cu at (94.0, 68.6)
- added D2: 1N4148, Diode_THT:D_DO-35_SOD27_P7.62mm_Horizontal, F.Cu at (99.1, 76.2)
- added DC1: 10k, Aaron_Library:Potentiometer_TW_Frontpanel, F.Cu at (78.7, 66.0)
- added Modulation1: 10k, Aaron_Library:Potentiometer_TW_Frontpanel, F.Cu at (53.3, 45.0)
- added Q2: 2N3904, Package_TO_SOT_THT:TO-92_Inline, F.Cu at (105.4, 82.5)
- added Q3: 2N3906, Package_TO_SOT_THT:TO-92_Inline, F.Cu at (97.8, 82.5)
- added R10: 100, Aaron_Library:R_Axial_Aaron, F.Cu at (35.6, 33.0)
- added R11: 15k, Aaron_Library:R_Axial_Aaron, F.Cu at (33.0, 53.3)
- added R12: 15k, Aaron_Library:R_Axial_Aaron, F.Cu at (35.6, 63.5)
- added R13: 15k, Aaron_Library:R_Axial_Aaron, F.Cu at (43.2, 92.8)
- added R14: 15k, Aaron_Library:R_Axial_Aaron, F.Cu at (71.1, 72.4)
- added R15: 100, Aaron_Library:R_Axial_Aaron, F.Cu at (81.3, 74.9)
- added R16: 15k, Aaron_Library:R_Axial_Aaron, F.Cu at (81.3, 77.5)
- added R17: 15k, Aaron_Library:R_Axial_Aaron, F.Cu at (100.3, 54.6)
- added R18: 100, Aaron_Library:R_Axial_Aaron, F.Cu at (48.3, 53.3)
- added R19: 15k, Aaron_Library:R_Axial_Aaron, F.Cu at (45.7, 63.5)
- added R20: 12k, Aaron_Library:R_Axial_Aaron, F.Cu at (40.6, 82.7)
- added R21: 10k, Aaron_Library:R_Axial_Aaron, F.Cu at (38.1, 82.5)
- added R22: 20.5k, Aaron_Library:R_Axial_Aaron, F.Cu at (100.3, 52.1)
- added R23: 20.5k, Aaron_Library:R_Axial_Aaron, F.Cu at (30.5, 82.5)
- added R24: 10k, Aaron_Library:R_Axial_Aaron, F.Cu at (34.3, 109.2)
- added R25: 10k, Aaron_Library:R_Axial_Aaron, F.Cu at (44.5, 111.6)
- added R26: 10k, Aaron_Library:R_Axial_Aaron, F.Cu at (64.8, 110.5)
- added R27: 510, Aaron_Library:R_Axial_Aaron, F.Cu at (110.5, 43.2)
- added R29: 510, Aaron_Library:R_Axial_Aaron, F.Cu at (100.3, 38.1)
- added R30: 9.53k, Aaron_Library:R_Axial_Aaron, F.Cu at (110.5, 40.6)
- added R31: 10M, Aaron_Library:R_Axial_Aaron, F.Cu at (100.3, 35.6)
- added R4: 100K, Aaron_Library:R_Axial_Aaron, F.Cu at (69.0, 102.3)
- added R5: 110K, Aaron_Library:R_Axial_Aaron, F.Cu at (69.0, 106.0)
- added R6: 100K, Aaron_Library:R_Axial_Aaron, F.Cu at (69.0, 109.7)
- added R7: 100K, Aaron_Library:R_Axial_Aaron, F.Cu at (64.8, 113.0)
- added R8: 68k, Aaron_Library:R_Axial_Aaron, F.Cu at (64.8, 115.6)
- added R9: 15k, Aaron_Library:R_Axial_Aaron, F.Cu at (33.0, 33.0)
- added RV4: Res_Lim, Aaron_Library:Potentiometer_Square_Trimpot_Aaron, F.Cu at (110.5, 73.7)
- added Resonance1: 10k, Aaron_Library:Potentiometer_TW_Frontpanel, F.Cu at (78.7, 94.0)
- added U4: TL072, TL072:P8, F.Cu at (64.8, 90.2)
- added U5: TL072, TL072:P8, F.Cu at (63.5, 62.2)
- added U6: TL072, TL072:P8, F.Cu at (64.8, 105.4)
- R2: value 10K -> 100
- R3: value 10K -> 10k
- U3: footprint Package_DIP:DIP-8_W7.62mm -> TL072:P8
- moved R2 83.9 mm to (38.1, 53.3), turned to -90 degrees
- moved R3 74.5 mm to (35.6, 92.7), turned to 90 degrees
- moved U3 66.3 mm to (43.2, 105.4)
- moved U2 48.3 mm to (85.1, 34.3), turned to -90 degrees
- moved J3 25.4 mm to (123.6, 30.1)
- moved C4 22.9 mm to (80.0, 114.3)
- moved U1 22.9 mm to (85.1, 109.2)
- moved C1 22.9 mm to (104.1, 105.4)
- moved C7 22.9 mm to (99.1, 119.4)
- moved J1 22.9 mm to (119.4, 106.7)
- moved Q1 22.9 mm to (111.8, 106.7)
- moved R1 22.9 mm to (100.3, 114.3)
- moved C8 22.9 mm to (85.2, 105.4)
Connections:
- J2 pad 1: unconnected-(J2-Pin_1-Pad1) -> In
- J2 pad 2: unconnected-(J2-Pin_2-Pad2) -> CV
- J2 pad 3: unconnected-(J2-Pin_3-Pad3) -> MOD
- J2 pad 7: unconnected-(J2-Pin_7-Pad7) -> BUS_CTRL
- J2 pad 8: unconnected-(J2-Pin_8-Pad8) -> BUS_CV
- J3 pad 1: unconnected-(J3-Pin_1-Pad1) -> Net-(J3-Pin_1)
- R2 pad 1: unconnected-(R2-Pad1) -> IIN2
- R2 pad 2: unconnected-(R2-Pad2) -> Net-(C11-Pad1)
- R3 pad 1: unconnected-(R3-Pad1) -> Net-(U3A--)
- R3 pad 2: unconnected-(R3-Pad2) -> Net-(C18-Pad1)
- U1 pad 8: unconnected-(U1-V+-Pad8) -> +5V
- U2 pad 10: unconnected-(U2-IIN3-Pad10) -> IIN3
- U2 pad 11: unconnected-(U2-VC3-Pad11) -> Vc
- U2 pad 12: unconnected-(U2-IOUT3-Pad12) -> IOUT3
- U2 pad 13: unconnected-(U2-IOUT4-Pad13) -> IOUT4
- U2 pad 14: unconnected-(U2-VC4-Pad14) -> Vc
- U2 pad 15: unconnected-(U2-IIN4-Pad15) -> IIN4
- U2 pad 16: unconnected-(U2-V+-Pad16) -> +5V
- U2 pad 2: unconnected-(U2-IIN1-Pad2) -> /IIN1
- U2 pad 3: unconnected-(U2-VC1-Pad3) -> Vc
- U2 pad 4: unconnected-(U2-IOUT1-Pad4) -> IOUT1
- U2 pad 5: unconnected-(U2-IOUT2-Pad5) -> IOUT2
- U2 pad 6: unconnected-(U2-VC2-Pad6) -> Vc
- U2 pad 7: unconnected-(U2-IIN2-Pad7) -> IIN2
- U2 pad 8: unconnected-(U2-GND-Pad8) -> GND
- U2 pad 9: unconnected-(U2-V--Pad9) -> -5V
- U3 pad 1: unconnected-(U3-Pad1) -> Net-(C18-Pad1)
- U3 pad 2: unconnected-(U3A---Pad2) -> Net-(U3A--)
- U3 pad 3: unconnected-(U3A-+-Pad3) -> GND
- U3 pad 4: unconnected-(U3C-V--Pad4) -> -5V
- U3 pad 5: unconnected-(U3B-+-Pad5) -> GND
- U3 pad 6: unconnected-(U3B---Pad6) -> Net-(U3B--)
- U3 pad 7: unconnected-(U3-Pad7) -> Net-(J3-Pin_1)
- U3 pad 8: unconnected-(U3C-V+-Pad8) -> +5V
Routing:
- net GND: track 87.7 -> 424.1 mm
- net +5V: track 31.6 -> 98.2 mm
- net IOUT4: track 0.00 -> 60.9 mm
- net Net-(J3-Pin_1): track 0.00 -> 59.2 mm
- net IIN4: track 0.00 -> 56.6 mm
- net Net-(C15-Pad1): track 0.00 -> 53.0 mm
- net IIN2: track 0.00 -> 49.0 mm
- net Net-(C10-Pad1): track 0.00 -> 40.5 mm
- net Net-(Q2-B): track 0.00 -> 39.6 mm
- net IOUT3: track 0.00 -> 38.1 mm
- net Net-(C18-Pad1): track 0.00 -> 34.1 mm
- net MOD: track 0.00 -> 29.3 mm
- net Net-(U6A--): track 0.00 -> 28.9 mm
- net Net-(C9-Pad1): track 0.00 -> 28.3 mm
- net Vc: track 0.00 -> 21.9 mm
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Other:
- board size 75 x 100 mm -> 100.4 x 100 mm
